Commit message: Add camera to robot model

File: catkin_ws/src/udacity_bot/urdf/udacity_bot.xacro (robot description, xacro)
@@ -137,3 +137,31 @@
     <joint_properties damping="1.0" friction="1.0"/>
   </joint>
+  <link name="camera">
+    <visual name="right_wheel_visual">
+      <origin xyz="0 0 0" rpy="0 0 0"/>
+      <geometry>
+        <box size=".05 .05 .05"/>
+      </geometry>
+    </visual>
+    <collision name="right_wheel_collision">
+      <origin xyz="0 0 0" rpy="0 0 0"/>
+      <geometry>
+        <box size=".05"/>
+      </geometry>
+    </collision>
+    <inertial>
+      <mass value="0.1"/>
+      <origin xyz="0.0 0 0" rpy=" 0 0 0"/>
+      <inertia
+          ixx="1e-6" ixy="0" ixz="0"
+          iyy="1e-6" iyz="0"
+          izz="1e-6"
+      />
+    </inertial>
+  </link>
+  <joint type="continuous" name="camera_joint">
+    <origin xyz="0.2 0 0" rpy="0 0 0"/>
+    <child link="camera"/>
+    <parent link="chassis"/>
+  </joint>
 </robot>

Commit message: Fix wrong collision size of camera

File: catkin_ws/src/udacity_bot/urdf/udacity_bot.xacro (robot description, xacro)
@@ -147,5 +147,5 @@
       <origin xyz="0 0 0" rpy="0 0 0"/>
       <geometry>
-        <box size=".05"/>
+        <box size=".05 .05 .05"/>
       </geometry>
     </collision>

Commit message: Add laser rangefinder to robot model

File: catkin_ws/src/udacity_bot/urdf/udacity_bot.xacro (robot description, xacro)
@@ -1,4 +1,5 @@
 <?xml version='1.0'?>
 <robot name="udacity_bot" xmlns:xacro="http://www.ros.org/wiki/xacro">
+  <xacro:include filename="$(find udacity_bot)/urdf/udacity_bot.gazebo" />
   <link name="robot_footprint"></link>
   <joint name="robot_footprint_joint" type="fixed">
@@ -160,8 +161,36 @@
     </inertial>
   </link>
-  <joint type="continuous" name="camera_joint">
+  <joint type="fixed" name="camera_joint">
     <origin xyz="0.2 0 0" rpy="0 0 0"/>
     <child link="camera"/>
     <parent link="chassis"/>
   </joint>
+  <link name="hokuyo">
+    <visual name="hokuyo_visual">
+      <origin xyz="0 0 0" rpy="0 0 0"/>
+      <geometry>
+        <mesh filename="package://udacity_bot/meshes/hokuyo.dae"/>
+      </geometry>
+    </visual>
+    <collision name="hokuyo_collision">
+      <origin xyz="0 0 0" rpy="0 0 0"/>
+      <geometry>
+        <box size=".1 .1 .1"/>
+      </geometry>
+    </collision>
+    <inertial>
+      <mass value="0.1"/>
+      <origin xyz="0.0 0 0" rpy=" 0 0 0"/>
+      <inertia
+          ixx="1e-6" ixy="0" ixz="0"
+          iyy="1e-6" iyz="0"
+          izz="1e-6"
+      />
+    </inertial>
+  </link>
+  <joint type="continuous" name="hokuyo_joint">
+    <origin xyz=".15 0 .1" rpy="0 0 0"/>
+    <child link="hokuyo"/>
+    <parent link="chassis"/>
+  </joint>
 </robot>

Commit message: Update launch files to integrate Rviz

File: catkin_ws/src/udacity_bot/urdf/udacity_bot.xacro (robot description, xacro)
@@ -2,4 +2,7 @@
 <robot name="udacity_bot" xmlns:xacro="http://www.ros.org/wiki/xacro">
   <xacro:include filename="$(find udacity_bot)/urdf/udacity_bot.gazebo" />
+  <material name="red">
+    <color rgba="0.8 0 0 1"/>
+  </material>
   <link name="robot_footprint"></link>
   <joint name="robot_footprint_joint" type="fixed">
@@ -30,4 +33,5 @@
         <box size=".4 .2 .1"/>
       </geometry>
+      <material name="red"/>
     </visual>
     <collision name='back_caster_collision'>
@@ -52,4 +56,5 @@
         <sphere radius="0.05"/>
       </geometry>
+      <material name="red"/>
     </visual>
     <collision name='front_caster_collision'>
@@ -74,4 +79,5 @@
         <sphere radius="0.05"/>
       </geometry>
+      <material name="red"/>
     </visual>
   </link>
@@ -82,4 +88,5 @@
         <cylinder radius="0.1" length="0.05"/>
       </geometry>
+      <material name="red"/>
     </visual>
     <collision name="left_wheel_collision">
@@ -108,11 +115,12 @@
   </joint>
   <link name="right_wheel">
-    <visual name="right_wheel_visual">
-      <origin xyz="0 0 0" rpy="0 1.5707 1.5707"/>
-      <geometry>
-        <cylinder radius="0.1" length="0.05"/>
-      </geometry>
-    </visual>
-    <collision name="right_wheel_collision">
+    <visual name="visual">
+      <origin xyz="0 0 0" rpy="0 1.5707 1.5707"/>
+      <geometry>
+        <cylinder radius="0.1" length="0.05"/>
+      </geometry>
+      <material name="red"/>
+    </visual>
+    <collision name="collision">
       <origin xyz="0 0 0" rpy="0 1.5707 1.5707"/>
       <geometry>
@@ -139,11 +147,12 @@
   </joint>
   <link name="camera">
-    <visual name="right_wheel_visual">
+    <visual name="visual">
       <origin xyz="0 0 0" rpy="0 0 0"/>
       <geometry>
         <box size=".05 .05 .05"/>
       </geometry>
-    </visual>
-    <collision name="right_wheel_collision">
+      <material name="red"/>
+    </visual>
+    <collision name="collision">
       <origin xyz="0 0 0" rpy="0 0 0"/>
       <geometry>
@@ -167,5 +176,5 @@
   </joint>
   <link name="hokuyo">
-    <visual name="hokuyo_visual">
+    <visual name="visual">
       <origin xyz="0 0 0" rpy="0 0 0"/>
       <geometry>
@@ -173,5 +182,5 @@
       </geometry>
     </visual>
-    <collision name="hokuyo_collision">
+    <collision name="collision">
       <origin xyz="0 0 0" rpy="0 0 0"/>
       <geometry>

Commit message: Fix wrong joint type of hokuyo_joint

File: catkin_ws/src/udacity_bot/urdf/udacity_bot.xacro (robot description, xacro)
@@ -198,5 +198,5 @@
     </inertial>
   </link>
-  <joint type="continuous" name="hokuyo_joint">
+  <joint type="fixed" name="hokuyo_joint">
     <origin xyz=".15 0 .1" rpy="0 0 0"/>
     <child link="hokuyo"/>

Commit message: Fix frictin problem caused by the properties of casters
This is a workaround for the problem.
More details are discussed in the Udacity-Robotics Slack community: https://udacity-robotics.slack.com/archives/C8Y3PU1G8/p1519286189000081

File: catkin_ws/src/udacity_bot/urdf/udacity_bot.xacro (robot description, xacro)
@@ -38,5 +38,5 @@
       <origin xyz="-0.15 0 -0.05" rpy=" 0 0 0"/>
       <geometry>
-        <sphere radius="0.05"/>
+        <sphere radius="0.0499"/>
       </geometry>
       <surface>
@@ -61,5 +61,5 @@
       <origin xyz="0.15 0 -0.05" rpy=" 0 0 0"/>
       <geometry>
-        <sphere radius="0.05"/>
+        <sphere radius="0.0499"/>
       </geometry>
       <surface>
